Commit message: Insert intermediate link and update joints

File: rrr_description/urdf/rrr.xacro (robot description, xacro)
@@ -243,7 +243,32 @@
     </gazebo>
     <joint name="joint_3" type="revolute">
-        <origin xyz="${radius_3 + radius_4} 0.0 ${length_3 - radius_3}" rpy="0.0 0.0 0.0" />
+        <origin xyz="${radius_3 + radius_3} 0.0 ${length_3 - radius_3}" rpy="0.0 0.0 0.0" />
         <parent link="link_2" />
         <child link="link_3" />
+        <axis xyz="1.0 0.0 0.0" />
+        <limit lower="0.0" upper="${M_PI * 2}" effort="300.0" velocity="1.0" />
+    </joint>
+    <!--link_3-->
+    <link name="link_3">
+        <xacro:inertial_block mass="${mass_3}" length="${length_3}" radius="${radius_3}" />
+        <visual>
+            <origin xyz="0.0 0.0 ${length_3/2.0}" rpy="0.0 0.0 0.0" />
+            <geometry>
+                <cylinder radius="${radius_3}" length="${length_3}" />
+            </geometry>
+            <material name="Grey" />
+        </visual>
+        <collision>
+            <origin xyz="0.0 0.0 ${length_3/2.0}" rpy="0.0 0.0 0.0" />
+            <geometry>
+                <cylinder radius="${radius_3}" length="${length_3}" />
+            </geometry>
+        </collision>
+    </link>
+    <xacro:gazebo_grey_link_color_block link_name="link_3" />
+    <joint name="joint_4" type="revolute">
+        <origin xyz="${radius_3 + radius_4} 0.0 ${length_3 - radius_3}" rpy="0.0 0.0 0.0" />
+        <parent link="link_3" />
+        <child link="link_4" />
         <axis xyz="1.0 0.0 0.0" />
         <limit lower="0.0" upper="${M_PI * 2}" effort="300.0" velocity="1.0" />
@@ -267,15 +292,15 @@
         </collision>
     </link>
-    <xacro:gazebo_grey_link_color_block link_name="link_3" />
-    <joint name="joint_4" type="revolute">
+    <xacro:gazebo_grey_link_color_block link_name="link_4" />
+    <joint name="joint_5" type="revolute">
         <origin xyz="0.0 0.0 ${length_4}" rpy="0.0 0.0 0.0" />
-        <parent link="link_3" />
-        <child link="link_4" />
-        <axis xyz="0.0 0.0 01.0" />
-        <limit lower="0.0" upper="${M_PI * 2}" effort="300.0" velocity="1.0" />
-    </joint>
-    <!--=============================================================================-->
-    <!--link_4-->
-    <link name="link_4">
+        <parent link="link_4" />
+        <child link="link_5" />
+        <axis xyz="0.0 0.0 1.0" />
+        <limit lower="0.0" upper="${M_PI * 2}" effort="300.0" velocity="1.0" />
+    </joint>
+    <!--=============================================================================-->
+    <!--link_5-->
+    <link name="link_5">
         <xacro:inertial_block mass="${mass_5}" length="${length_5}" radius="${radius_5}" />
         <visual>
@@ -293,8 +318,8 @@
         </collision>
     </link>
-    <xacro:gazebo_grey_link_color_block link_name="link_4" />
+    <xacro:gazebo_grey_link_color_block link_name="link_5" />
     <joint name="gripper_joint_1" type="prismatic">
         <origin xyz="0.0 0.0 ${radius_5 + length_6/2.0}" rpy="0.0 0.0 0.0" />
-        <parent link="link_4" />
+        <parent link="link_5" />
         <child link="gripper_link_1" />
         <axis xyz="1.0 0.0 0.0" />
@@ -303,5 +328,5 @@
     <joint name="gripper_joint_2" type="prismatic">
         <origin xyz="0.0 0.0 ${radius_5 + length_6/2.0}" rpy="0.0 0.0 0.0" />
-        <parent link="link_4" />
+        <parent link="link_5" />
         <child link="gripper_link_2" />
         <axis xyz="1.0 0.0 0.0" />
@@ -310,5 +335,5 @@
     <joint name="gripper_frame_joint" type="fixed">
         <origin xyz="0.0 0.0 ${radius_5*2 + length_6/2 + 0.01}" rpy="0.0 0.0 0.0" />
-        <parent link="link_4" />
+        <parent link="link_5" />
         <child link="gripper_frame_cp" />
     </joint>

File: rrr_description/urdf/rrr_control.xacro (robot description, xacro)
@@ -35,4 +35,11 @@
             <state_interface name="position" />
         </joint>
+        <joint name="joint_5">
+            <command_interface name="position">
+                <param name="min">0.0</param>
+                <param name="max">6.28</param>
+            </command_interface>
+            <state_interface name="position" />
+        </joint>
         <joint name="gripper_joint_1">
             <command_interface name="position">
